File: HelloFOC.kicad_sch (KiCad schematic)
At the start: 61 parts, among them J1 USB-C, J2 Motor, J3 Debug, J4 Encoder, Q1 Q_NMOS_GSD, Q2 Q_NMOS_GSD, Q3 Q_NMOS_GSD, Q4 Q_NMOS_GSD, Q5 Q_NMOS_GSD, Q6 Q_NMOS_GSD, SW1 BOOT, U1 SPX3819M5-L-3-3, U2 ESP32-C3-MINI-1, U3 XL6019E1, U4 ME3116, U5 FD6288Q

Commit message: Finish BOM
Parts:
- C1, C12, C13, C14, C16, C17, C18, C2, C20, C21, C22, C4, C6: footprint (none) -> Capacitor_SMD:C_0402_1005Metric
- C10, C11, C7, C8, C9: footprint (none) -> Capacitor_SMD:C_1206_3216Metric
- C15, C19, C5: footprint (none) -> Capacitor_SMD:C_0402_1005Metric; Manufacturer (none) -> SAMSUNG; PartNumber (none) -> C307331; Supplier (none) -> JLC
- C3: value 10uF -> 10nF; footprint (none) -> Capacitor_SMD:C_0402_1005Metric
- D1: value D_Schottky -> SS34; footprint (none) -> Diode_SMD:D_SMC; Manufacturer (none) -> LGE; PartNumber (none) -> C717457; Supplier (none) -> JLC-EXT
- D2, D3, D4, D5: value D_Schottky -> B5819WS; footprint (none) -> Diode_SMD:D_SOD-323; Manufacturer (none) -> Slkor; PartNumber (none) -> C488405; Supplier (none) -> JLC-EXT
- J1: footprint (none) -> JLC-SMT:HRO_TYPE-C-31-M-12; Manufacturer (none) -> HRO; PartNumber (none) -> C165948; Supplier (none) -> JLC-EXT
- J2: Manufacturer (none) -> TXGA; PartNumber (none) -> C2834021; Supplier (none) -> JLC-EXT
- J3: footprint (none) -> Connector_PinHeader_2.54mm:PinHeader_1x02_P2.54mm_Vertical
- J4: Manufacturer (none) -> kinghelm; PartNumber (none) -> C709364; Supplier (none) -> JLC-EXT
- L1: footprint (none) -> Inductor_SMD:L_10.4x10.4_H4.8; Manufacturer (none) -> COILMX; PartNumber (none) -> C380056; Supplier (none) -> JLC-EXT
- L2: footprint (none) -> Inductor_SMD:L_1008_2520Metric; Manufacturer (none) -> COILMX; PartNumber (none) -> C435291; Supplier (none) -> JLC-EXT
- Q1, Q2, Q3, Q4, Q5, Q6: value Q_NMOS_GSD -> EMB09N03V; footprint (none) -> JLC-SMT:EMC_EMB09N03V; symbol Device:Q_NMOS_GSD -> Device:Q_NMOS_SGD; Manufacturer (none) -> EMC; PartNumber (none) -> C461957; Supplier (none) -> JLC-EXT
- R1, R10, R11, R12, R13, R14, R15, R16, R2, R3, R4, R5, R6, R7, R8, R9: footprint (none) -> Resistor_SMD:R_0402_1005Metric
- SW1: footprint (none) -> JLC-SMT:SMD-SW-4_5.1X5.1; Manufacturer (none) -> XKB; PartNumber (none) -> C318884; Supplier (none) -> JLC
- U1: Manufacturer (none) -> MaxLinear; PartNumber (none) -> C9055; Supplier (none) -> JLC-EXT
- U2: Manufacturer (none) -> ESPRESSIF; PartNumber (none) -> C2838502; Supplier (none) -> JLC-EXT
- U3: Manufacturer (none) -> XLSEMI; PartNumber (none) -> C73018; Supplier (none) -> JLC-EXT
- U4: Manufacturer (none) -> MICRONE; PartNumber (none) -> C97643; Supplier (none) -> JLC-EXT
- U5: Manufacturer (none) -> Fortior Tech; PartNumber (none) -> C328453; Supplier (none) -> JLC-EXT
Connections:
- net GND: now also Q4.1 (S), Q5.1 (S), Q6.1 (S); no longer Q4.2 (S), Q5.2 (S), Q6.2 (S)
- net HO_A: now also Q1.2 (G); no longer Q1.1 (G)
- net HO_B: now also Q2.2 (G); no longer Q2.1 (G)
- net HO_C: now also Q3.2 (G); no longer Q3.1 (G)
- net LO_A: now also Q4.2 (G); no longer Q4.1 (G)
- net LO_B: now also Q5.2 (G); no longer Q5.1 (G)
- net LO_C: now also Q6.2 (G); no longer Q6.1 (G)
- net MOTOR_A: now also Q1.1 (S); no longer Q1.2 (S)
- net MOTOR_B: now also Q2.1 (S); no longer Q2.2 (S)
- net MOTOR_C: now also Q3.1 (S); no longer Q3.2 (S)
